File: deskamp.kicad_pcb (KiCad board)
At the start: 2 copper layers, 34 parts, among them J1 Input 01, J10 Input Select, J2 Input 02, J3 Preamp Out, J5 LFE, J6 Mute, J7 Sleep, J8 Motor, J9 Power, K1 TQ2-12V, K2 TQ2-12V, K3 TQ2-12V, K4 TQ2-12V, Q1 PN2222A, Q2 PN2222A, Q3 PN2222A, Q4 PN2222A, U1 esp32-wemos-d1-mini, U2 L9110, U3 TSR_1-2433

Commit message: Update deskamp.kicad_pcb
Routing:
- net GND: track 262.2 -> 272.4 mm
Changed lines of the file:
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@@
+	)
+	(segment
+		(start 163.6 94.55)
+		(end 163.6 88.55)
+		(width 1)
+		(layer "B.Cu")
+		(net 11)
 	)
 	(segment
@@
 	)
 	(segment
+		(start 170.15 101.1)
+		(end 163.6 94.55)
+		(width 1)
+		(layer "B.Cu")
+		(net 11)
+	)
+	(segment
+		(start 176.245 101.1)
+		(end 170.15 101.1)
+		(width 1)
+		(layer "B.Cu")
+		(net 11)
+	)
+	(segment
 		(start 169.755 121.76)
 		(end 176.245 115.27)
@@
 		(layer "B.Cu")
 		(net 11)
-	)
-	(segment
-		(start 176.245 101.1)
-		(end 168.35 93.205)
-		(width 1)
-		(layer "B.Cu")
-		(net 11)

Commit message: Switch motor gpio for board layout
Connections:
- U2 pad 6: Net-(U1-IO_04) -> Net-(U1-IO_00)
- U2 pad 7: Net-(U1-IO_00) -> Net-(U1-IO_04)
Changed lines of the file:
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@@
 			(layers "*.Cu" "*.Mask")
 			(remove_unused_layers no)
-			(net 35 "Net-(U1-IO_04)")
+			(net 52 "Net-(U1-IO_00)")
 			(pinfunction "IA")
 			(pintype "input")
@@
 			(layers "*.Cu" "*.Mask")
 			(remove_unused_layers no)
-			(net 52 "Net-(U1-IO_00)")
+			(net 35 "Net-(U1-IO_04)")
 			(pinfunction "IB")
 			(pintype "input")
