File: esp32-preamp.kicad_pcb (KiCad board)
At the start: 2 copper layers, 126 x 68 mm, 49 parts, among them J1 INPUT 1, J10 LFE, J11 OUT, J2 INPUT 2, J3 AMP PWR, J5 VOLUME, J6 TSOP382, J7 SELECT, J8 POT MOTOR, J9 PWR IN, Q1 2N3904, Q2 2N3904, Q3 2N3904, U3 TSR0.5-2450, U4 TLV702475DBV, U5 TPS60402DBV, U6 ESP32 D1 Mini, U7 TPS72301DBV

Commit message: PGA2311
Parts:
- removed C10, C12: 2.2uF, Capacitor_SMD:C_1206_3216Metric_Pad1.33x1.80mm_HandSolder
- removed C9: 1uF, Capacitor_SMD:C_1206_3216Metric_Pad1.33x1.80mm_HandSolder
- R8: moved to B.Cu
- moved R11 104.7 mm to (108.3, 167.0), turned to 180 degrees
- moved R10 104.1 mm to (108.3, 163.0), turned to 180 degrees
- moved R9 103.6 mm to (108.3, 159.0), turned to 180 degrees
- moved J5 96.8 mm to (132.8, 163.1)
- moved J7 79.9 mm to (118.6, 163.0)
- moved C8 64.5 mm to (32.3, 70.7), turned to 90 degrees
- moved J8 57.2 mm to (40.0, 54.8)
- moved U2 50.3 mm to (37.0, 73.6)
- moved C7 48.9 mm to (121.5, 120.5), turned to 180 degrees
- moved U6 31.0 mm to (92.5, 102.2), turned to 0 degrees
- moved U3 28.9 mm to (60.5, 103.8), turned to 0 degrees
- moved J6 22.7 mm to (30.4, 94.1)
- moved J9 18.5 mm to (61.8, 92.9)
- moved C1 16.7 mm to (138.8, 125.7)
- moved C3 16.6 mm to (166.5, 133.0)
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Connections:
- J10 pad 1: GNDA -> Net-(J10-Pin_1)
- J10 pad 2: Net-(J10-Pin_2) -> GNDA
- J11 pad 1: GNDA -> Net-(J11-Pin_1)
- J11 pad 3: Net-(J11-Pin_3) -> GNDA
- R5 pad 1: Net-(J11-Pin_3) -> Net-(J11-Pin_2)
- R5 pad 2: Net-(J10-Pin_2) -> Net-(J10-Pin_1)
- R6 pad 1: Net-(J11-Pin_2) -> Net-(J11-Pin_1)
- R6 pad 2: Net-(J10-Pin_2) -> Net-(J10-Pin_1)
- U1 pad 11: Net-(J11-Pin_2) -> Net-(J11-Pin_1)
- U1 pad 14: Net-(J11-Pin_3) -> Net-(J11-Pin_2)
- U4 pad 3: +5VD -> unconnected-(U4-EN-Pad3)
Routing:
- net Net-(J11-Pin_1): track 0.00 -> 56.6 mm
- net Net-(J11-Pin_2): track 0.00 -> 55.8 mm
- net +12V: track 27.0 -> 72.9 mm
- net IN_L: track 0.00 -> 38.1 mm
- net IN_R: track 0.00 -> 38.1 mm
- net Net-(J10-Pin_1): track 0.00 -> 24.6 mm
- net GNDA: track 0.00 -> 17.5 mm, vias 0 -> 2
- net -5VA: track 30.4 -> 14.4 mm
- net GNDD: track 0.00 -> 12.5 mm, vias 0 -> 4
- net Net-(Q1-B): track 0.00 -> 9.45 mm
- net Net-(U5-C_{FLY-}): track 0.00 -> 8.04 mm
- net +5VA: track 22.7 -> 15.2 mm
- net Net-(Q2-B): track 0.00 -> 7.05 mm
- net Net-(Q3-B): track 0.00 -> 6.10 mm
- net Net-(U5-C_{FLY+}): track 0.00 -> 4.99 mm
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Other:
- board text added: "+"
- board text added: "+3.3V"
- board text added: "01"
- board text added: "02"
- board text added: "03"
- board text added: "ADC"
- board text added: "COM"
- board text added: "DATA"
- board text added: "GND"
- board text added: "L"
- board text added: "R"
